Commit message: Add nav2, use laserscan for grid map, and adjust camera angle so it's now without 15 degree tilt

File: src/my_create_map_webots/resource/MyCreate_kinect.urdf (robot description, URDF)
Before this commit: robot /home/jordenhuang/ROS2-Project/src/my_create_map_webots/resource/MyCreate_kinect_.urdf, 25 links, 24 joints
Joints:
- joint base_to_kinect_joint: origin xyz=0.14 0 0.10 rpy=0 0.261799 0 -> xyz=0.14 0 0.10 rpy=0 0 0
