Commit message: Rename my_create_map_webots to my_create_simulation

File: src/my_create_simulation/resource/MyCreate.urdf (robot description, URDF)
Before this commit: robot /home/jordenhuang/ROS2-Project/src/my_create_map_webots/resource/MyCreate_kinect_.urdf, 25 links, 24 joints
Links:
- removed link Kinect
- removed link camera_depth_frame
- removed link camera_depth_optical_frame
- removed link camera_rgb_frame
- removed link camera_rgb_optical_frame
- added link base_footprint
- added link camera_left
- added link camera_left_optical_frame
- added link camera_right
- added link camera_right_optical_frame
Joints:
- removed joint base_to_kinect_joint
- removed joint camera_depth_to_camera_depth_optical_joint
- removed joint camera_rgb_to_camera_rgb_optical_joint
- removed joint kinect_to_camera_depth_joint
- removed joint kinect_to_camera_rgb_joint
- added joint base_joint: type fixed, parent base_link, child base_footprint, origin xyz=0 0 -0.05 rpy=0 0 0
- added joint base_link_camera_left_joint: type fixed, parent base_link, child camera_left, origin xyz=0.17 0.05 0.05 rpy=0.0 0.261799 0.0
- added joint base_link_camera_right_joint: type fixed, parent base_link, child camera_right, origin xyz=0.17 -0.05 0.05 rpy=0.0 0.261799 0.0
- added joint camera_left_to_optical_joint: type fixed, parent camera_left, child camera_left_optical_frame, origin xyz=0 0 0 rpy=-1.570796 0 -1.570796
- added joint camera_right_to_optical_joint: type fixed, parent camera_right, child camera_right_optical_frame, origin xyz=0 0 0 rpy=-1.570796 0 -1.570796
- joint base_link_bumper_left_joint: origin xyz=0 0 0 rpy=1.570806 0.000006 -0.843867 -> xyz=0 0 -0.000003 rpy=1.570806 0.000006 -0.843867
- joint base_link_bumper_right_joint: origin xyz=0 0 0 rpy=1.570792 0.000011 -2.297729 -> xyz=0 0 -0.000003 rpy=1.570792 0.000011 -2.297729
- joint left wheel motor: origin xyz=-0.0062 0 -0.014 rpy=0 0 0 -> xyz=-0.0062 0 -0.014 rpy=0 -0.000002 0
- joint right wheel motor: origin xyz=-0.0062 0.1359 -0.014 rpy=0 0 0 -> xyz=-0.0062 0.1359 -0.014 rpy=0 -0.000002 0

File: src/my_create_simulation/resource/MyCreate_kinect.urdf (robot description, URDF)
Before this commit: robot /home/jordenhuang/ROS2-Project/src/my_create_map_webots/resource/MyCreate_realsense.urdf, 34 links, 33 joints
Links:
- removed link MPU-9250
- removed link MPU-9250 accelerometer
- removed link MPU-9250 compass
- removed link MPU-9250 gyro
- removed link Realsense
- removed link RealsenseD455_display
- removed link RealsenseD455_emitter
- removed link RealsenseD455_receiver
- removed link imu_link
- removed link solid
- added link Kinect; collision box size=0.084 0.027 0.068; visual box size=0.084 0.027 0.068
- link base_link: geometry 
Joints:
- removed joint MPU-9250_MPU-9250 accelerometer_joint
- removed joint MPU-9250_MPU-9250 compass_joint
- removed joint MPU-9250_MPU-9250 gyro_joint
- removed joint MPU9250_to_imu_link_joint
- removed joint base_link_MPU-9250_joint
- removed joint base_link_RealsenseD455_display_joint
- removed joint base_link_RealsenseD455_emitter_joint
- removed joint base_link_RealsenseD455_receiver_joint
- removed joint base_link_solid_joint
- removed joint base_to_realsense_joint
- removed joint realsense_to_camera_depth_joint
- removed joint realsense_to_camera_rgb_joint
- added joint base_to_kinect_joint: type fixed, parent base_link, child Kinect, origin xyz=0.14 0 0.10 rpy=0 0 0
- added joint kinect_to_camera_depth_joint: type fixed, parent Kinect, child camera_depth_frame, origin xyz=0 0 0 rpy=0 0 0
- added joint kinect_to_camera_rgb_joint: type fixed, parent Kinect, child camera_rgb_frame, origin xyz=0 0 0 rpy=0 0 0

File: src/my_create_simulation/resource/MyCreate_realsense.urdf (robot description, URDF)
Before this commit: robot /home/jordenhuang/ROS2-Project/src/my_create_map_webots/resource/MyCreate.urdf, 25 links, 24 joints
Links:
- removed link base_footprint
- removed link camera_left
- removed link camera_left_optical_frame
- removed link camera_right
- removed link camera_right_optical_frame
- added link MPU-9250
- added link MPU-9250 accelerometer
- added link MPU-9250 compass
- added link MPU-9250 gyro
- added link Realsense; collision box size=0.084 0.027 0.068; visual box size=0.084 0.027 0.068
- added link RealsenseD455_display
- added link RealsenseD455_emitter
- added link RealsenseD455_receiver
- added link camera_depth_frame
- added link camera_depth_optical_frame
- added link camera_rgb_frame
- added link camera_rgb_optical_frame
- added link imu_link
- added link solid
- link base_link: geometry collision box size=0.027 0.123 0.025; visual box size=0.027 0.123 0.025
Joints:
- removed joint base_joint
- removed joint base_link_camera_left_joint
- removed joint base_link_camera_right_joint
- removed joint camera_left_to_optical_joint
- removed joint camera_right_to_optical_joint
- added joint MPU-9250_MPU-9250 accelerometer_joint: type fixed, parent MPU-9250, child MPU-9250 accelerometer, origin xyz=0 0 0 rpy=0 0 0
- added joint MPU-9250_MPU-9250 compass_joint: type fixed, parent MPU-9250, child MPU-9250 compass, origin xyz=0 0 0 rpy=0 0 0
- added joint MPU-9250_MPU-9250 gyro_joint: type fixed, parent MPU-9250, child MPU-9250 gyro, origin xyz=0 0 0 rpy=0 0 0
- added joint MPU9250_to_imu_link_joint: type fixed, parent MPU-9250, child imu_link, origin xyz=0 0 0 rpy=0 0 0
- added joint base_link_MPU-9250_joint: type fixed, parent base_link, child MPU-9250, origin xyz=0.15 0 0.05 rpy=0 0 0
- added joint base_link_RealsenseD455_display_joint: type fixed, parent base_link, child RealsenseD455_display, origin xyz=0 0 0 rpy=0 0 0
- added joint base_link_RealsenseD455_emitter_joint: type fixed, parent base_link, child RealsenseD455_emitter, origin xyz=0 0 0 rpy=0 0 0
- added joint base_link_RealsenseD455_receiver_joint: type fixed, parent base_link, child RealsenseD455_receiver, origin xyz=0 0 0 rpy=0 0 0
- added joint base_link_solid_joint: type fixed, parent base_link, child solid, origin xyz=0.013 0 0 rpy=1.570798 -0.000002 1.570801
- added joint base_to_realsense_joint: type fixed, parent base_link, child Realsense, origin xyz=0.14 0 0.05 rpy=0 0 0
- added joint camera_depth_to_camera_depth_optical_joint: type fixed, parent camera_depth_frame, child camera_depth_optical_frame, origin xyz=0 0 0 rpy=-1.570796 0 -1.570796
- added joint camera_rgb_to_camera_rgb_optical_joint: type fixed, parent camera_rgb_frame, child camera_rgb_optical_frame, origin xyz=0 0 0 rpy=-1.570796 0 -1.570796
- added joint realsense_to_camera_depth_joint: type fixed, parent Realsense, child camera_depth_frame, origin xyz=0.005 0 0 rpy=0 0 0
- added joint realsense_to_camera_rgb_joint: type fixed, parent Realsense, child camera_rgb_frame, origin xyz=0.005 0 0 rpy=0 0 0
- joint base_link_bumper_left_joint: origin xyz=0 0 -0.000003 rpy=1.570806 0.000006 -0.843867 -> xyz=0 0 0 rpy=1.570806 0.000006 -0.843867
- joint base_link_bumper_right_joint: origin xyz=0 0 -0.000003 rpy=1.570792 0.000011 -2.297729 -> xyz=0 0 0 rpy=1.570792 0.000011 -2.297729
- joint left wheel motor: origin xyz=-0.0062 0 -0.014 rpy=0 -0.000002 0 -> xyz=-0.0062 0 -0.014 rpy=0 0 0
- joint right wheel motor: origin xyz=-0.0062 0.1359 -0.014 rpy=0 -0.000002 0 -> xyz=-0.0062 0.1359 -0.014 rpy=0 0 0
