Commit message: Remove "backup" behavior in nav2

File: src/my_create/resource/create_with_realsense.urdf.xacro (robot description, xacro)
@@ -8,5 +8,5 @@
   <xacro:include filename="$(find realsense2_description)/urdf/_d435i.urdf.xacro"/>
   <xacro:sensor_d435i parent="base_link" use_nominal_extrinsics="false">
-    <origin xyz="0.5 0 0.14" rpy="0 0 0"/>
+    <origin xyz="0.15 0 0.05" rpy="0 0 0"/>
   </xacro:sensor_d435i>
     <!-- <joint name="base_link_to_camera_link_joint" type="fixed">
